File: kicad/opamp-vos.kicad_pcb (KiCad board)
At the start: 2 copper layers, 49.5 x 49.5 mm, 38 parts, among them P1 CONN_01X02, Q1 2N3904, Q2 2N3904, Q3 2N3904, Q4 2N3904, U1 7805, U2 TL074, U3 TL072, U4 TL071

Commit message: working on v2 board layout
Parts:
- removed 1PIN (x5): P***, PL_mounting_holes:1pin_05_09
- removed C1: 10uF, PL_capacitors:ELCAP_10_20_V_059A
- removed C3: 0.1uF, PL_capacitors:CERCAP_2_059B_0805
- removed D1, D2, D3, D4, D5: LED, PL_LEDs:LED_3MM_069A
- removed D6: 1N4001, PL_diodes:DIODE_1A_069A_PL
- removed G***: OSHW-logo_silkscreen-front_4mm, OSHW-logo:OSHW-logo_silkscreen-front_4mm
- removed the H*** at (163.8, 109.2)
- removed the H*** at (121.9, 109.2)
- removed the H*** at (163.8, 67.3)
- removed the H*** at (121.9, 67.3)
- removed P1: CONN_01X02, PL_connectors:BARREL_JACK_21x55
- removed Q1, Q2, Q3, Q4: 2N3904, PL_TO-92:TO-92_Q_EBC_059Bo_PL
- removed R1: 100k, PL_resistors:R_AXIAL_0W25_059A_PL
- removed R2: 47k, PL_resistors:R_AXIAL_0W25_059A_PL
- removed R3, R6, R7: 220, PL_resistors:R_AXIAL_0W25_059A_PL
- removed R4, R5, R8, R9: 1k, PL_resistors:R_AXIAL_0W25_059A_PL
- removed U1: 7805, PL_TO-220:TO-220_V_069A
- removed U2: TL074, PL_DIP:DIP14_PL
- removed U3: TL072, PL_DIP:DIP8_059A_PL
- removed U4: TL071, PL_DIP:DIP8_059A_PL
- added C10: 0.1uF, CERCAP_15_059B_0805, F.Cu at (146.7, 81.3)
- added C11: 0.1uF, CERCAP_15_059B_0805, F.Cu at (152.4, 94.0)
- added C12: 10nF, CERCAP_15_059B_0805, F.Cu at (149.9, 94.0)
- added C20: 0.1uF, CERCAP_15_059B_0805, F.Cu at (169.5, 81.3)
- added C21: 0.1uF, CERCAP_15_059B_0805, F.Cu at (175.3, 94.0)
- added C22: 10nF, CERCAP_15_059B_0805, F.Cu at (172.7, 94.0)
- added C30: 0.1uF, CERCAP_15_059B_0805, F.Cu at (95.9, 63.5)
- added C31: 0.1uF, CERCAP_15_059B_0805, F.Cu at (95.9, 66.7)
- added C32: 0.1uF, CERCAP_15_059B_0805, F.Cu at (90.2, 63.5)
- added C33: 0.1uF, CERCAP_15_059B_0805, F.Cu at (90.2, 66.7)
- added C40: 0.1uF, CERCAP_15_059B_0805, F.Cu at (278.1, 99.1)
- added C41: 0.1uF, CERCAP_15_059B_0805, F.Cu at (270.5, 93.3)
- added C42: 0.1uF, CERCAP_15_059B_0805, F.Cu at (272.4, 108.6)
- added C43: 0.1uF, CERCAP_15_059B_0805, F.Cu at (245.7, 85.7)
- added C44: 0.1uF, CERCAP_15_059B_0805, F.Cu at (263.5, 86.4)
- added C45: 0.1uF, CERCAP_15_059B_0805, F.Cu at (254.0, 86.4)
- added C60: 1uF, ELCAP_10_20_V_059A, F.Cu at (182.2, 151.8)
- added C61: 1uF, ELCAP_10_20_V_059A, F.Cu at (182.2, 173.4)
- added C62: 0.1uF, CERCAP_15_059B_0805, F.Cu at (189.2, 161.9)
- added C63: 0.1uF, CERCAP_15_059B_0805, F.Cu at (186.1, 165.7)
- added CON60: BARREL_JACK, BARREL_JACK_21x55, F.Cu at (181.0, 143.5)
- added D60: 1N4148, DIODE_SS_059A_03_PL, F.Cu at (184.8, 143.5)
- added D61: 1N4148, DIODE_SS_059A_03_PL, F.Cu at (177.2, 160.0)
- added D62: 1N4148, DIODE_SS_059A_03_PL, F.Cu at (177.2, 167.6)
- added H***: Val**, hole_M3, F.Cu at (268.0, 134.0)
- added H***: Val**, hole_M3, F.Cu at (268.0, 177.2)
- added H***: Val**, hole_M3, F.Cu at (174.6, 177.2)
- added H***: Val**, hole_M3, F.Cu at (174.6, 134.0)
- added JP10: JUMPER, SIL-2, F.Cu at (146.7, 78.1)
- added JP11: JUMPER, SIL-2, F.Cu at (153.0, 78.1)
- added JP20: JUMPER, SIL-2, F.Cu at (178.4, 78.1)
- added JP21: JUMPER, SIL-2, F.Cu at (172.1, 78.1)
- added P60: CONN_2X1, SIL-2, F.Cu at (172.7, 151.1)
- added Q60: 2N3904, TO-92_Q_EBC_059Bo_PL, F.Cu at (188.6, 158.1)
- added Q61: 2N3906, TO-92_Q_EBC_059Bo_PL, F.Cu at (187.3, 169.5)
- added R12: 10, R_AXIAL_0W25_059A_PL, F.Cu at (146.1, 104.1)
- added R13: 10k, R_AXIAL_0W25_059A_PL, F.Cu at (146.1, 101.6)
- added R14: 10k, 3296W_PL, F.Cu at (151.1, 73.7)
- added R15: 0R, R_AXIAL_0W25_059A_PL, F.Cu at (156.2, 69.2)
- added R20: 10k, R_AXIAL_0W25_059A_PL, F.Cu at (179.1, 96.5)
- added R21: 10, R_AXIAL_0W25_059A_PL, F.Cu at (168.9, 99.1)
- added R22: 10, R_AXIAL_0W25_059A_PL, F.Cu at (168.9, 101.6)
- added R23: 10k, R_AXIAL_0W25_059A_PL, F.Cu at (168.9, 104.1)
- added R24: 20k, 3296W_PL, F.Cu at (174.0, 73.7)
- added R25: 0R, R_AXIAL_0W25_059A_PL, F.Cu at (168.9, 69.2)
- added R30: 10k, R_AXIAL_0W25_059A_PL, F.Cu at (89.5, 80.0)
- added R31: 10, R_AXIAL_0W25_059A_PL, F.Cu at (89.5, 82.5)
- added R32: 10, R_AXIAL_0W25_059A_PL, F.Cu at (89.5, 85.1)
- added R33: 10k, R_AXIAL_0W25_059A_PL, F.Cu at (89.5, 87.6)
- added R35: 10k, R_AXIAL_0W25_059A_PL, F.Cu at (89.5, 90.2)
- added R36: 10, R_AXIAL_0W25_059A_PL, F.Cu at (89.5, 92.7)
- added R37: 10, R_AXIAL_0W25_059A_PL, F.Cu at (89.5, 95.2)
- added R38: 10k, R_AXIAL_0W25_059A_PL, F.Cu at (89.5, 97.8)
- added R40: 10k, R_AXIAL_0W25_059A_PL, F.Cu at (251.5, 89.5)
- added R41: 10, R_AXIAL_0W25_059A_PL, F.Cu at (251.5, 92.1)
- added R42: 10, R_AXIAL_0W25_059A_PL, F.Cu at (251.5, 94.6)
- added R43: 10k, R_AXIAL_0W25_059A_PL, F.Cu at (251.5, 97.2)
- added R44: 10k, R_AXIAL_0W25_059A_PL, F.Cu at (251.5, 99.7)
- added R45: 10, R_AXIAL_0W25_059A_PL, F.Cu at (251.5, 102.2)
- added R46: 10, R_AXIAL_0W25_059A_PL, F.Cu at (251.5, 104.8)
- added R47: 10k, R_AXIAL_0W25_059A_PL, F.Cu at (251.5, 107.3)
- added R48: 10k, R_AXIAL_0W25_059A_PL, F.Cu at (251.5, 109.9)
- added R49: 10, R_AXIAL_0W25_059A_PL, F.Cu at (251.5, 112.4)
- added R50: 10, R_AXIAL_0W25_059A_PL, F.Cu at (251.5, 114.9)
- added R51: 10k, R_AXIAL_0W25_059A_PL, F.Cu at (251.5, 117.5)
- added R52: 10k, R_AXIAL_0W25_059A_PL, F.Cu at (251.5, 120.0)
- added R53: 10, R_AXIAL_0W25_059A_PL, F.Cu at (251.5, 122.6)
- added R54: 10, R_AXIAL_0W25_059A_PL, F.Cu at (251.5, 125.1)
- added R55: 10k, R_AXIAL_0W25_059A_PL, F.Cu at (251.5, 127.6)
- added R60: 4.7k, R_AXIAL_0W25_059A_PL, F.Cu at (173.4, 157.5)
- added R61: 4.7k, R_AXIAL_0W25_059A_PL, F.Cu at (183.5, 170.2)
- added R62: 10R, R_AXIAL_0W25_059A_PL, F.Cu at (183.5, 162.6)
- added R63: 10R, R_AXIAL_0W25_059A_PL, F.Cu at (173.4, 165.1)
- added TP0: TEST, TEST, F.Cu at (188.0, 177.2)
- added TP11: TEST, TEST, F.Cu at (158.1, 87.6)
- added TP12: TEST, TEST, F.Cu at (147.3, 66.0)
- added TP13: TEST, TEST, F.Cu at (151.1, 66.0)
- added TP14: TEST, TEST, F.Cu at (154.9, 66.0)
- added TP21: TEST, TEST, F.Cu at (181.0, 87.6)
- added TP22: TEST, TEST, F.Cu at (177.8, 66.0)
- added TP23: TEST, TEST, F.Cu at (174.0, 66.0)
- added TP24: TEST, TEST, F.Cu at (170.2, 66.0)
- added TP31: TEST, TEST, F.Cu at (95.9, 101.0)
- added TP32: TEST, TEST, F.Cu at (91.4, 101.0)
- added TP41: TEST, TEST, F.Cu at (268.6, 82.5)
- added TP42: TEST, TEST, F.Cu at (268.6, 75.6)
- added TP43: TEST, TEST, F.Cu at (268.6, 78.7)
- added TP44: TEST, TEST, F.Cu at (268.6, 72.4)
- added U10: UA741, DIP8_059A_PL, F.Cu at (147.3, 91.4)
- added U20: OP07, DIP8_059A_PL, F.Cu at (170.2, 91.4)
- added U30: LM358, DIP8_059A_PL, F.Cu at (90.8, 76.8)
- added U40: LM324, DIP14_PL, F.Cu at (248.9, 82.5)
- R10: value 220 -> 10k; footprint PL_resistors:R_AXIAL_0W25_059A_PL -> R_AXIAL_0W25_059A_PL
- R11: value 220 -> 10; footprint PL_resistors:R_AXIAL_0W25_059A_PL -> R_AXIAL_0W25_059A_PL
- moved R10 16.0 mm to (156.2, 96.5), turned to 180 degrees
- moved R11 5.75 mm to (146.1, 99.1)
Connections:
- R10 pad 1: 5V -> Vos1
- R10 pad 2: Net-(D3-Pad1) -> N-0000027
- R11 pad 1: 5V -> N-0000027
- R11 pad 2: Net-(D4-Pad1) -> Vgnd
Routing:
- net 5V: track 138.2 -> 0.00 mm
- net LED1: track 93.6 -> 0.00 mm, vias 2 -> 0
- net Vee: track 0.00 -> 92.2 mm
- net LED2: track 86.5 -> 0.00 mm, vias 8 -> 0
- net 1.6V: track 81.9 -> 0.00 mm
- net Vcc: track 0.00 -> 54.6 mm
- net LED4: track 41.6 -> 0.00 mm, vias 2 -> 0
- net LED3: track 41.3 -> 0.00 mm, vias 4 -> 0
- net N-0000023: track 0.00 -> 25.9 mm
- net Vos1: track 0.00 -> 18.7 mm
- net Vos2: track 0.00 -> 17.0 mm
- net N-000008: track 0.00 -> 16.2 mm
- net N-0000033: track 0.00 -> 15.9 mm
- net N-0000011: track 0.00 -> 15.7 mm
- net N-000006: track 0.00 -> 15.7 mm
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- added copper zone on B.Cu, net Vgnd
- removed copper zone on B.Cu, net GND
Other:
- board size 49.5 x 49.5 mm -> 99.7 x 49.5 mm
- net class Default: clearance 0.2 -> 0.254; trace_width 0.25 -> 0.254; via_dia 0.6 -> 0.889; via_drill 0.4 -> 0.635
- rule pad_to_mask_clearance: 0.2 -> 0
- rule trace_clearance: 0.2 -> 0.254
- rule trace_min: 0.2 -> 0.254
- rule via_min_drill: 0.3 -> 0.508
- rule via_min_size: 0.4 -> 0.889
- board text removed: "(v1)"
- board text removed: "LM324"
- board text removed: "LM358"
- board text removed: "LM741"
- board text removed: "NE5532"
- board text removed: "NE5534"
- board text removed: "Opamp Input Offset Voltage Tester"
- board text removed: "POWER (9V)"
- board text removed: "TL071"
- board text removed: "TL072"
- board text removed: "TL074"
- board text removed: "VOS1"
- board text removed: "VOS2"
- board text removed: "VOS3"
- board text removed: "VOS4"
- board text removed: "VREF"
- board text removed: "github.com/pepaslabs/opamp-vos"

Commit message: working on v2 board layout
Parts:
- moved R32 164.8 mm to (253.4, 102.9), turned to 270 degrees
- moved C31 164.1 mm to (255.9, 102.9), turned to 270 degrees
- moved R38 164.0 mm to (253.4, 90.2), turned to 90 degrees
- moved R33 162.0 mm to (250.8, 102.9), turned to 270 degrees
- moved R37 161.4 mm to (250.8, 90.2), turned to 90 degrees
- moved R31 160.0 mm to (248.3, 102.9), turned to 270 degrees
- moved R36 158.8 mm to (248.3, 90.2), turned to 90 degrees
- moved C32 158.5 mm to (243.2, 104.8), turned to 270 degrees
- moved R30 157.9 mm to (245.7, 102.9), turned to 270 degrees
- moved U30 156.7 mm to (245.7, 100.3)
- moved R35 156.2 mm to (245.7, 90.2), turned to 90 degrees
- moved C33 154.1 mm to (243.2, 84.5), turned to 90 degrees
- moved TP32 151.3 mm to (242.6, 94.6)
- moved C30 149.7 mm to (243.2, 90.2), turned to 90 degrees
- moved TP31 146.7 mm to (242.6, 98.4)
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Routing:
- net N-0000013: track 0.00 -> 18.8 mm
- net N-0000019: track 0.00 -> 18.8 mm
- net N-0000022: track 0.00 -> 18.8 mm
- net N-0000041: track 0.00 -> 17.7 mm
- net N-000004: track 0.00 -> 17.3 mm
- net N-0000042: track 0.00 -> 16.9 mm
- net Vos3B: track 0.00 -> 10.1 mm
- net Vos4B: track 0.00 -> 7.56 mm
- net Vos4C: track 0.00 -> 7.56 mm
- net Vos4A: track 0.00 -> 7.56 mm
- net Vos4D: track 0.00 -> 7.56 mm
- net Vos3A: track 0.00 -> 6.50 mm
- net Vcc: track 54.6 -> 60.7 mm
- net Vee: track 92.2 -> 98.3 mm
- net N-000003: track 0.00 -> 5.08 mm
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