File: kicad/opamp-vos.kicad_pcb (KiCad board)
At the start: 2 copper layers, 99.7 x 49.5 mm, 94 parts, among them CON60 BARREL_JACK, P60 CONN_2X1, Q60 2N3904, Q61 2N3906, U10 UA741, U20 OP07, U30 LM358, U40 LM324

Commit message: v2 gerbers
Parts:
- added G***: OSHW-logo_silkscreen-front_6mm, OSHW-logo_silkscreen-front_6mm, F.Cu at (184.8, 134.0)
- added R16: 0R, R_AXIAL_0W25_059A_PL, F.Cu at (193.7, 142.9)
- added R17: 0R, R_AXIAL_0W25_059A_PL, F.Cu at (193.7, 145.4)
- added R26: 0R, R_AXIAL_0W25_059A_PL, F.Cu at (219.7, 142.9)
- added R27: 0R, R_AXIAL_0W25_059A_PL, F.Cu at (219.7, 145.4)
- U10: value UA741 -> uA741
- moved R15 8.26 mm to (203.8, 148.0)
- moved R25 8.26 mm to (209.6, 148.0)
- moved R14 5.72 mm to (198.8, 138.4), turned to 0 degrees
- moved R24 5.72 mm to (214.6, 138.4), turned to 0 degrees
- moved C20 4.58 mm to (209.6, 154.3), turned to 0 degrees
- moved TP12 4.58 mm to (198.8, 134.0)
- moved TP13 4.58 mm to (194.9, 134.0)
- moved C10 2.54 mm to (194.3, 154.3)
- moved R11 2.54 mm to (193.7, 172.1)
- moved R21 2.54 mm to (209.6, 172.1)
- moved C11 2.54 mm to (200.0, 167.0)
- moved C12 2.54 mm to (197.5, 167.0)
- moved C21 2.54 mm to (215.9, 167.0)
- moved C22 2.54 mm to (213.4, 167.0)
- moved JP10 2.54 mm to (194.3, 151.1)
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Connections:
- JP10 pad 1: N-0000033 (its old number) -> N-0000035
- JP11 pad 1: N-0000034 (its old number) -> N-0000036
- JP20 pad 1: N-000008 -> N-0000016
- JP21 pad 1: N-000005 (its old number) -> N-000008
- R14 pad 1: N-0000034 (its old number) -> N-0000015
- R14 pad 3: N-0000033 (its old number) -> N-0000010
- R24 pad 1: N-000008 -> N-0000017
- R24 pad 3: N-000005 (its old number) -> N-000009
- TP12 pad 1: N-0000033 (its old number) -> N-0000035
- TP14 pad 1: N-0000034 (its old number) -> N-0000036
- TP22 pad 1: N-000008 -> N-0000016
- TP24 pad 1: N-000005 (its old number) -> N-000008
Routing:
- net N-0000035: track 0.00 -> 23.3 mm
- net N-0000016: track 0.00 -> 20.4 mm
- net N-0000036: track 0.00 -> 20.0 mm
- net N-0000033 (its old number): track 15.9 -> 0.00 mm
- net N-000005 (its old number): track 12.9 -> 0.00 mm
- net N-0000034 (its old number): track 12.9 -> 0.00 mm
- net N-0000015: track 0.00 -> 9.46 mm
- net N-0000045: track 12.3 -> 21.5 mm
- net N-0000017: track 0.00 -> 9.09 mm
- net Vee: track 274.2 -> 265.4 mm
- net N-000008: track 16.2 -> 22.2 mm
- net N-000009: track 0.00 -> 5.50 mm
- net N-0000010: track 0.00 -> 5.50 mm
- net Vcc: track 202.9 -> 207.3 mm
- net N-000007: track 12.3 -> 16.1 mm
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Other:
- board text added: "LT1001"
- board text added: "NE5532"
- board text added: "NE5534"
- board text added: "Op Amp Vos Tester"
- board text added: "TL061"
- board text added: "TL062"
- board text added: "TL064"
- board text added: "VGND"
- board text added: "Vcc"
- board text added: "Vee"
- board text added: "Vos"
- board text added: "Vos1"
- board text added: "Vos2"
- board text added: "Vos3"
- board text added: "Vos4"
- board text added: "https://www.github.com/pepaslabs/opamp-vos"
- board text added: "v2"
- board text removed: "+"
- board text removed: "-"

Commit message: v2 gerbers
Other:
- outline, holes or cut-outs redrawn
- board text added: "PIN1"
- board text added: "PIN5"
- board text added: "PIN8"
- board text added: "TAP"
Changed lines of the file:
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@@
     (links 160)
     (no_connects 0)
-    (area 171.399999 130.759999 271.195001 180.390001)
+    (area 166.895779 129.158999 272.796001 181.991001)
     (thickness 1.6)
-    (drawings 24)
+    (drawings 34)
     (tracks 277)
     (zones 0)
@@
     (visible_elements FFFFFFBF)
     (pcbplotparams
-      (layerselection 3178497)
+      (layerselection 284196865)
       (usegerberextensions true)
       (excludeedgelayer true)
@@
       (outputformat 1)
       (mirror false)
-      (drillshape 1)
+      (drillshape 0)
       (scaleselection 1)
-      (outputdirectory ""))
+      (outputdirectory gerbers))
   )
   (net 0 "")
@@
     (tags "CONN DEV")
     (fp_text reference TP24 (at 0 1.905 180) (layer F.SilkS)
-      (effects (font (size 0.635 0.635) (thickness 0.127)))
+      (effects (font (size 0.762 0.762) (thickness 0.1524)))
     )
     (fp_text value TEST (at 0 -1.905 180) (layer F.SilkS) hide
@@
     (tags "CONN DEV")
     (fp_text reference TP22 (at 0 1.905 180) (layer F.SilkS)
-      (effects (font (size 0.635 0.635) (thickness 0.127)))
+      (effects (font (size 0.762 0.762) (thickness 0.1524)))
     )
     (fp_text value TEST (at 0 -1.905 180) (layer F.SilkS) hide
@@
     (tags "CONN DEV")
     (fp_text reference TP23 (at 0 1.905 180) (layer F.SilkS)
-      (effects (font (size 0.635 0.635) (thickness 0.127)))
+      (effects (font (size 0.762 0.762) (thickness 0.1524)))
     )
     (fp_text value TEST (at 0 -1.905 180) (layer F.SilkS) hide
@@
     (tags "CONN DEV")
     (fp_text reference TP12 (at 0 1.905 180) (layer F.SilkS)
-      (effects (font (size 0.635 0.635) (thickness 0.127)))
+      (effects (font (size 0.762 0.762) (thickness 0.1524)))
     )
     (fp_text value TEST (at 0 -1.905 180) (layer F.SilkS) hide
@@
     (tags "CONN DEV")
     (fp_text reference TP13 (at 0 1.905 180) (layer F.SilkS)
-      (effects (font (size 0.635 0.635) (thickness 0.127)))
+      (effects (font (size 0.762 0.762) (thickness 0.1524)))
     )
     (fp_text value TEST (at 0 -1.905 180) (layer F.SilkS) hide
@@
     (tags "CONN DEV")
     (fp_text reference TP14 (at 0 1.905 180) (layer F.SilkS)
-      (effects (font (size 0.635 0.635) (thickness 0.127)))
+      (effects (font (size 0.762 0.762) (thickness 0.1524)))
     )
     (fp_text value TEST (at 0 -1.905 180) (layer F.SilkS) hide
@@
       (xy -1.81864 2.69494)) (layer F.SilkS) (width 0.00254))
   )
+  (gr_arc (start 267.97 133.985) (end 267.97 130.81) (angle 90) (layer Edge.Cuts) (width 0.1))
+  (gr_arc (start 267.97 177.165) (end 271.145 177.165) (angle 90) (layer Edge.Cuts) (width 0.1))
+  (gr_arc (start 174.625 177.165) (end 174.625 180.34) (angle 90) (layer Edge.Cuts) (width 0.1))
+  (gr_arc (start 174.625 133.985) (end 171.45 133.985) (angle 90) (layer Edge.Cuts) (width 0.1))
+  (gr_line (start 267.97 130.81) (end 174.625 130.81) (angle 90) (layer Edge.Cuts) (width 0.1))
+  (gr_line (start 271.145 133.985) (end 271.145 177.165) (angle 90) (layer Edge.Cuts) (width 0.1))
+  (gr_line (start 174.625 180.34) (end 267.97 180.34) (angle 90) (layer Edge.Cuts) (width 0.1))
+  (gr_text TAP (at 193.04 133.985 90) (layer F.SilkS)
+    (effects (font (size 0.762 0.762) (thickness 0.1524)))
+  )
+  (gr_text TAP (at 212.725 133.985 90) (layer F.SilkS)
+    (effects (font (size 0.762 0.762) (thickness 0.1524)))
+  )
+  (gr_text PIN8 (at 208.915 133.985 90) (layer F.SilkS)
+    (effects (font (size 0.762 0.762) (thickness 0.1524)))
+  )
+  (gr_text PIN1 (at 216.535 133.985 90) (layer F.SilkS)
+    (effects (font (size 0.762 0.762) (thickness 0.1524)))
+  )
+  (gr_text PIN5 (at 200.66 133.985 90) (layer F.SilkS)
+    (effects (font (size 0.762 0.762) (thickness 0.1524)))
+  )
+  (gr_text PIN1 (at 196.85 133.985 90) (layer F.SilkS)
+    (effects (font (size 0.762 0.762) (thickness 0.1524)))
+  )
+  (gr_line (start 171.45 133.985) (end 171.45 177.165) (angle 90) (layer Edge.Cuts) (width 0.1))
   (gr_text Vos3 (at 267.335 153.67 270) (layer F.SilkS)
     (effects (font (size 0.762 0.762) (thickness 0.1524)))
@@
     (effects (font (size 1.016 1.016) (thickness 0.2032)) (justify left))
   )
-  (gr_line (start 171.45 180.34) (end 171.45 130.81) (angle 90) (layer Edge.Cuts) (width 0.1))
-  (gr_line (start 271.145 180.34) (end 171.45 180.34) (angle 90) (layer Edge.Cuts) (width 0.1))
-  (gr_line (start 271.145 130.81) (end 271.145 180.34) (angle 90) (layer Edge.Cuts) (width 0.1))
-  (gr_line (start 171.45 130.81) (end 271.145 130.81) (angle 90) (layer Edge.Cuts) (width 0.1))
   (segment (start 252.095 161.925) (end 252.095 159.385) (width 0.254) (layer F.Cu) (net 1))
   (segment (start 249.555 161.925) (end 252.095 161.925) (width 0.254) (layer F.Cu) (net 1))

Commit message: v2.1
Parts:
- U10: value uA741 -> UA741
Connections:
- C60 pad 2: Vgnd -> N-0000032
- C61 pad 1: Vgnd -> N-0000032
- D61 pad 2: Vgnd -> N-0000032
- D62 pad 1: Vgnd -> N-0000032
Routing:
- net N-0000032: track 0.00 -> 31.7 mm
Other:
- board text added: "v2.1"
- board text removed: "v2"
