File: kicad/opamp-vos.sch (KiCad schematic (older format))
At the start: 28 parts, among them P1 CONN_01X02, Q1 2N3904, Q2 2N3904, Q3 2N3904, Q4 2N3904, U1 7805, U2 TL074, U3 TL072, U4 TL071

Commit message: working on revision 2
Parts:
- removed C1: 10uF, PL_capacitors:ELCAP_10_20_V_059A, symbol C_EL
- removed C3: 0.1uF, PL_capacitors:CERCAP_2_059B_0805, symbol C_CER
- removed D1, D2, D3, D4, D5: LED, PL_LEDs:LED_3MM_069A, symbol LED
- removed D6: 1N4001, PL_diodes:DIODE_1A_069A_PL, symbol DIODE
- removed P1: CONN_01X02, PL_connectors:BARREL_JACK_21x55, symbol CONN_01X02
- removed Q1, Q2, Q3, Q4: 2N3904, PL_TO-92:TO-92_Q_EBC_059Bo_PL, symbol 2N3904
- removed R1: 100k, PL_resistors:R_AXIAL_0W25_059A_PL, symbol R_0W25
- removed R2: 47k, PL_resistors:R_AXIAL_0W25_059A_PL, symbol R_0W25
- removed R3, R6, R7: 220, PL_resistors:R_AXIAL_0W25_059A_PL, symbol R_0W25
- removed R4, R5, R8, R9: 1k, PL_resistors:R_AXIAL_0W25_059A_PL, symbol R_0W25
- removed U1: 7805, PL_TO-220:TO-220_V_069A, symbol 7805
- removed U2: TL074, PL_DIP:DIP14_PL, symbol TL074
- removed U3: TL072, PL_DIP:DIP8_059A_PL, symbol TL072
- removed U4: TL071, PL_DIP:DIP8_059A_PL, symbol TL071
- added C10, C11, C20, C21, C30, C31, C32, C33, C40, C41, C42, C43, C44, C45, C? (x6): 0.1uF, symbol C_CER
- added C12, C22: 10nF, symbol C_CER
- added C? (x3): 1uF, PL_capacitors:ELCAP_10_20_V_059A, symbol C_EL
- added CON? (x2): BARREL_JACK, ~, symbol BARREL_JACK
- added D? (x4): 1N4148, ~, symbol DIODE
- added JP10, JP11, JP20, JP21: JUMPER, ~, symbol JUMPER
- added P? (x2): CONN_2X1, ~, symbol CONN_2X1
- added Q?: 2N3904, symbol 2N3904
- added Q?: 2N3906, symbol 2N3906
- added R12, R21, R22, R31, R32, R36, R37, R41, R42, R45, R46, R49, R50, R53, R54: 10, PL_resistors:R_AXIAL_0W25_059A_PL, symbol R_0W25
- added R13, R20, R23, R30, R33, R35, R38, R40, R43, R44, R47, R48, R51, R52, R55: 10k, PL_resistors:R_AXIAL_0W25_059A_PL, symbol R_0W25
- added R14, R?: 10k, ~, symbol POT_25T
- added R15, R25: 0R, PL_resistors:R_AXIAL_0W25_059A_PL, symbol R_0W25
- added R24: 20k, ~, symbol POT_25T
- added R? (x2): 4.7k, PL_resistors:R_AXIAL_0W25_059A_PL, symbol R_0W25
- added R? (x3): 10R, PL_resistors:R_AXIAL_0W25_059A_PL, symbol R_0W25
- added TP10, TP11, TP12, TP13, TP14, TP20, TP21, TP22, TP23, TP24: TEST, ~, symbol TEST
- added U10: UA741, ~, symbol UA741
- added U20: OP07, ~, symbol OP07
- added U3, U?: LM358, ~, symbol LM358
- added U4: LM324, ~, symbol LM324
- R10: value 220 -> 10k
- R11: value 220 -> 10
Connections:
- net labels added: Vcc, Vee, Vgnd, Vos, Vos1
- net labels removed: +V, 1.6V, 5V, LED1, LED2, LED3, LED4
- wire segments 85 -> 255
- no-connect marks 2 -> 0
Other:
- note added: "LM324, etc."
- note added: "LM358, TL062, etc."
- note added: "OP07, etc."
- note added: "http://www.analog.com/media/en/training-seminars/tutorials/MT-037.pdf"
- note added: "https://tangentsoft.net/elec/vgrounds.html"
- note added: "uA741, TL061, etc."

Commit message: schematic for v2
Parts:
- removed C? (x4): 0.1uF, symbol C_CER
- removed C?: 1uF, PL_capacitors:ELCAP_10_20_V_059A, symbol C_EL
- removed CON?: BARREL_JACK, ~, symbol BARREL_JACK
- removed D?: 1N4148, ~, symbol DIODE
- removed P?: CONN_2X1, ~, symbol CONN_2X1
- removed R?: 10R, PL_resistors:R_AXIAL_0W25_059A_PL, symbol R_0W25
- removed R?: 10k, ~, symbol POT_25T
- removed TP20: TEST, ~, symbol TEST
- removed U?: LM358, ~, symbol LM358
- added TP30, TP31, TP40, TP41, TP42, TP43: TEST, ~, symbol TEST
- gave numbers to parts that had none: 15
- renumbered TP21 to TP20
Connections:
- net labels added: Vos2, Vos3A, Vos3B, Vos4A, Vos4B, Vos4C, Vos4D
- net labels removed: Vos
- wire segments 255 -> 224
Other:
- note added: "See https://www.github.com/pepaslabs/opamp-vos"
- moved on the sheet: C10, C11, C12, C20, C21, C22, C30, C31, C32, C33, C40, C41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

Commit message: working on v2 board layout
Parts:
- renumbered TP10 to TP0, TP14 to TP13, TP13 to TP14, TP20 to TP21, TP23 to TP22, TP24 to TP23, TP22 to TP24, TP30 to TP31, TP31 to TP32, TP40 to TP41, TP41 to TP42, TP42 to TP43, TP43 to TP44, U3 to U30, U4 to U40
Connections:
- net labels removed: GND
Changed lines of the file:
@@
 Sheet 1 1
 Title ""
-Date "9 jun 2018"
+Date "10 jun 2018"
 Rev ""
 Comp ""
@@
 D7 76 E9 D2 33 A7 13 7F 96 43 AB 24 25 25 D5 35 34 46 DB 8B 7E E0 94 DF 01 1C 67 24 18 EF 55 8D
 65 C6 A3 3B 96 19 8F EE 58 66 3C BA 63 99 F1 E8 8E 65 C6 A3 3B 96 F9 1F 63 08 66 50 C8 05 91 2A
-00 00 00 00 49 45 4E 44 AE 42 60 82 92 $EndBitmap
+00 00 00 00 49 45 4E 44 AE 42 60 82 00 $EndBitmap
 EndData
 $EndBitmap
@@
 uA741, TL061, etc.
 $Comp
-L LM358 U3
+L LM358 U30
 U 1 1 5B1B986E
 P 21400 5350
-F 0 "U3" H 21450 5475 40  0000 L CNN
+F 0 "U30" H 21450 5475 40  0000 L CNN
 F 1 "LM358" H 21450 5225 40  0000 L CNN
 F 2 "~" H 21400 5350 50  0000 C CNN
@@
 LM358, TL062, etc.
 $Comp
-L LM358 U3
+L LM358 U30
 U 2 1 5B1B98F3
 P 21350 8450
-F 0 "U3" H 21400 8575 40  0000 L CNN
+F 0 "U30" H 21400 8575 40  0000 L CNN
 F 1 "LM358" H 21400 8325 40  0000 L CNN
 F 2 "~" H 21350 8450 50  0000 C CNN
@@
 	20450 8350 20450 8450
 Connection ~ 20700 8350
-$Comp
-L GND #PWR?
-U 1 1 5B1B992B
-P 20700 8950
-F 0 "#PWR?" H 20700 8700 50  0001 C CNN
-F 1 "GND" H 20700 8800 50  0000 C CNN
-F 2 "" H 20700 8950 50  0000 C CNN
-F 3 "" H 20700 8950 50  0000 C CNN
-	1    20700 8950
-	1    0    0    -1
-$EndComp
-$Comp
-L GND #PWR?
-U 1 1 5B1B9931
-P 20450 8950
-F 0 "#PWR?" H 20450 8700 50  0001 C CNN
-F 1 "GND" H 20450 8800 50  0000 C CNN
-F 2 "" H 20450 8950 50  0000 C CNN
-F 3 "" H 20450 8950 50  0000 C CNN
-	1    20450 8950
-	1    0    0    -1
-$EndComp
 Wire Wire Line
 	20450 8850 20450 8950
@@
 $EndComp
 $Comp
-L TEST TP13
+L TEST TP14
 U 1 1 5B1C375E
 P 12550 7650
-F 0 "TP13" V 12550 7650 40  0000 C CNN
+F 0 "TP14" V 12550 7650 40  0000 C CNN
 F 1 "TEST" V 12650 7650 40  0000 C CNN
 F 2 "~" H 12600 7600 60  0000 C CNN
@@
 $EndComp
 $Comp
-L TEST TP14
+L TEST TP13
 U 1 1 5B1C3769
 P 11800 7450
-F 0 "TP14" V 11800 7450 40  0000 C CNN
+F 0 "TP13" V 11800 7450 40  0000 C CNN
 F 1 "TEST" V 11900 7450 40  0000 C CNN
 F 2 "~" H 11850 7400 60  0000 C CNN
@@
 $EndComp
 $Comp
-L TEST TP10
+L TEST TP0
 U 1 1 5B1C377A
 P 13500 5750
-F 0 "TP10" V 13500 5750 40  0000 C CNN
+F 0 "TP0" V 13500 5750 40  0000 C CNN
 F 1 "TEST" V 13600 5750 40  0000 C CNN
 F 2 "~" H 13550 5700 60  0000 C CNN
@@
 Vgnd
 $Comp
-L TEST TP23
+L TEST TP22
 U 1 1 5B1C380D
 P 17000 5600
-F 0 "TP23" V 17000 5600 40  0000 C CNN
+F 0 "TP22" V 17000 5600 40  0000 C CNN
 F 1 "TEST" V 17100 5600 40  0000 C CNN
 F 2 "~" H 17050 5550 60  0000 C CNN
@@
 $EndComp
 $Comp
-L TEST TP22
+L TEST TP24
 U 1 1 5B1C3813
 P 17200 6550
-F 0 "TP22" V 17200 6550 40  0000 C CNN
+F 0 "TP24" V 17200 6550 40  0000 C CNN
 F 1 "TEST" V 17300 6550 40  0000 C CNN
 F 2 "~" H 17250 6500 60  0000 C CNN
@@
 $EndComp
 $Comp
-L TEST TP24
+L TEST TP23
 U 1 1 5B1C3819
 P 17450 6200
-F 0 "TP24" V 17450 6200 40  0000 C CNN
+F 0 "TP23" V 17450 6200 40  0000 C CNN
 F 1 "TEST" V 17550 6200 40  0000 C CNN
 F 2 "~" H 17500 6150 60  0000 C CNN
@@
 $EndComp
 $Comp
-L TEST TP20
+L TEST TP21
 U 1 1 5B1C381F
 P 18150 7850
-F 0 "TP20" V 18150 7850 40  0000 C CNN
+F 0 "TP21" V 18150 7850 40  0000 C CNN
 F 1 "TEST" V 18250 7850 40  0000 C CNN
 F 2 "~" H 18200 7800 60  0000 C CNN
@@
 Vgnd
 $Comp
-L LM324 U4
+L LM324 U40
 U 1 1 5B1C5A07
 P 25600 5400
-F 0 "U4" H 25650 5525 40  0000 L CNN
+F 0 "U40" H 25650 5525 40  0000 L CNN
 F 1 "LM324" H 25650 5275 40  0000 L CNN
 F 2 "~" H 25600 5400 60  0000 C CNN
@@
 $EndComp
 $Comp
-L LM324 U4
+L LM324 U40
 U 2 1 5B1C5A23
 P 25550 8500
-F 0 "U4" H 25600 8625 40  0000 L CNN
+F 0 "U40" H 25600 8625 40  0000 L CNN
 F 1 "LM324" H 25600 8375 40  0000 L CNN
 F 2 "~" H 25550 8500 60  0000 C CNN
@@
 Vgnd
 $Comp
-L LM324 U4
+L LM324 U40
 U 3 1 5B1C5A7C
 P 25500 10850
-F 0 "U4" H 25550 10975 40  0000 L CNN
+F 0 "U40" H 25550 10975 40  0000 L CNN
 F 1 "LM324" H 25550 10725 40  0000 L CNN
 F 2 "~" H 25500 10850 60  0000 C CNN
@@
 Vgnd
 $Comp
-L LM324 U4
+L LM324 U40
 U 4 1 5B1C5ADC
 P 25500 13100
-F 0 "U4" H 25550 13225 40  0000 L CNN
+F 0 "U40" H 25550 13225 40  0000 L CNN
 F 1 "LM324" H 25550 12975 40  0000 L CNN
 F 2 "~" H 25500 13100 60  0000 C CNN
@@
 Vos3A
 $Comp
-L TEST TP30
+L TEST TP31
 U 1 1 5B1C77C7
 P 22650 5350
-F 0 "TP30" V 22650 5350 40  0000 C CNN
+F 0 "TP31" V 22650 5350 40  0000 C CNN
 F 1 "TEST" V 22750 5350 40  0000 C CNN
 F 2 "~" H 22700 5300 60  0000 C CNN
@@
 Connection ~ 22300 5350
 $Comp
-L TEST TP31
+L TEST TP32
 U 1 1 5B1C799C
 P 22700 8450
-F 0 "TP31" V 22700 8450 40  0000 C CNN
+F 0 "TP32" V 22700 8450 40  0000 C CNN
 F 1 "TEST" V 22800 8450 40  0000 C CNN
 F 2 "~" H 22750 8400 60  0000 C CNN
@@
 Vos4A
 $Comp
-L TEST TP40
+L TEST TP41
 U 1 1 5B1C7B73
 P 26800 5400
-F 0 "TP40" V 26800 5400 40  0000 C CNN
+F 0 "TP41" V 26800 5400 40  0000 C CNN
 F 1 "TEST" V 26900 5400 40  0000 C CNN
 F 2 "~" H 26850 5350 60  0000 C CNN
@@
 Connection ~ 26450 5400
 $Comp
-L TEST TP41
+L TEST TP42
 U 1 1 5B1C7D55
 P 26850 8500
-F 0 "TP41" V 26850 8500 40  0000 C CNN
+F 0 "TP42" V 26850 8500 40  0000 C CNN
 F 1 "TEST" V 26950 8500 40  0000 C CNN
 F 2 "~" H 26900 8450 60  0000 C CNN
@@
 $EndComp
 $Comp
-L TEST TP42
+L TEST TP43
 U 1 1 5B1C7D5B
 P 26850 10850
-F 0 "TP42" V 26850 10850 40  0000 C CNN
+F 0 "TP43" V 26850 10850 40  0000 C CNN
 F 1 "TEST" V 26950 10850 40  0000 C CNN
 F 2 "~" H 26900 10800 60  0000 C CNN
@@
 $EndComp
 $Comp
-L TEST TP43
+L TEST TP44
 U 1 1 5B1C7D61
 P 26800 13100
-F 0 "TP43" V 26800 13100 40  0000 C CNN
+F 0 "TP44" V 26800 13100 40  0000 C CNN
 F 1 "TEST" V 26900 13100 40  0000 C CNN
 F 2 "~" H 26850 13050 60  0000 C CNN
@@
 	26450 8300 26450 8500
 Connection ~ 26450 8500
+Text GLabel 20700 8950 3    40   Input ~ 0
+Vgnd
+Text GLabel 20450 8950 3    40   Input ~ 0
+Vgnd
 $EndSCHEMATC

Commit message: v2 gerbers
Parts:
- added R16, R17, R26, R27: 0R, PL_resistors:R_AXIAL_0W25_059A_PL, symbol R_0W25
Connections:
- wire segments 224 -> 228
Other:
- note added: "OP07, LT1001, NE5534, etc."
- note removed: "OP07, etc."
- moved on the sheet: C12, C20, R10, R11, R15, R25

Commit message: v2.1
Connections:
- wire segments 228 -> 227
Changed lines of the file:
@@
 LIBS:contrib
 LIBS:valves
+LIBS:opamp-vos-cache
 EELAYER 27 0
 EELAYER END
@@
 Sheet 1 1
 Title ""
-Date "10 jun 2018"
+Date "21 jun 2018"
 Rev ""
 Comp ""
@@
 22 70 21 48 58 23 70 21 48 58 23 70 21 48 58 23 70 21 48 58 23 70 21 48 58 23 70 21 48 58 23 70
 21 48 58 23 70 21 48 58 23 70 21 48 58 23 70 21 FF 03 38 BA 84 D5 3B 93 EB 94 00 00 00 00 49 45
-4E 44 AE 42 60 82 00 $EndBitmap
+4E 44 AE 42 60 82 FE $EndBitmap
 EndData
 $EndBitmap
@@
 06 83 19 9B 98 08 6D 84 A1 F0 FA 78 08 BC C2 50 9B 6B F0 63 C8 C7 83 1F 43 3E 1E FC 18 F2 F1 E0
 C7 90 8F 07 3F 86 7C 3C F8 31 E4 E3 C1 8F FF 03 9F 8A 64 AC E2 99 C6 EC 00 00 00 00 49 45 4E 44
-AE 42 60 82 13 $EndBitmap
+AE 42 60 82 FE $EndBitmap
 EndData
 $EndBitmap
@@
 Connection ~ 7050 10600
 Wire Wire Line
-	7700 9100 7050 9100
-Connection ~ 7050 9100
-Connection ~ 7700 9100
-Wire Wire Line
 	7050 9050 6600 9050
